Commit message: continued working on URDF file

File: src/arm_urdf/description/robot_core.xacro (robot description, xacro)
@@ -13,17 +13,50 @@
         <color rgba="0 0 0 1"/>
     </material>
-    <!-- SHOULDER LINK -->
+    <!-- BASE -->
     <link name="base_link">
     </link>
-    <joint name="base_to_shoulder" type="fixed">
+    <joint name="base_joint" type="fixed">
         <parent link ="base_link"/>
-        <child link="shoulder"/>
+        <child link="shoulder_link"/>
         <origin xyz="0 0 1"/>
     </joint>
-    <link name = "shoulder">
+    <!-- SHOULDER -->
+    <link name = "shoulder_link">
+        <visual>
+            <origin xyz="0 0 -0.05"/>
+            <geometry>
+                <box size="0.1 0.1 0.1"/>
+            </geometry>
+            <material name="blue"/>
+        </visual>
+    </link>
+    <joint name="shoulder_joint" type="revolute">
+        <parent link ="shoulder_link"/>
+        <child link="bicept_link"/>
+        <origin xyz="0 0 -0.1" rpy="0 0 0"/>
+        <axis xyz="0 1 0" rpy="0 0 0"/>
+        <limit lower="0" upper="${pi/2}" velocity ="100" effort = "100"/>
+    </joint>
+    <link name = "bicept_link">
+        <visual>
+            <origin xyz="0 0 0.5"/>
+            <geometry>
+                <box size="0.01 0.01 0.1"/>
+            </geometry>
+            <material name="orange"/>
+        </visual>
+    </link>
+    <joint name="bicept_joint" type="revolute">
+        <parent link ="bicept_link"/>
+        <child link="elbow_link"/>
+        <origin xyz="0 0 0.1" rpy="0 0 0"/>
+        <axis xyz="0 1 0" rpy="0 0 0"/>
+        <limit lower="0" upper="${pi/2}" velocity ="100" effort = "100"/>
+    </joint>
+    <link name = "elbow_link">
         <visual>
             <origin xyz="0 0 0.05"/>
             <geometry>
-                <box size="0.01 0.01 0.1"/>
+                <box size="0.1 0.11 0.1"/>
             </geometry>
             <material name="white"/>

Commit message: arm URDF V1

File: src/arm_urdf/description/robot_core.xacro (robot description, xacro)
@@ -18,26 +18,26 @@
     <joint name="base_joint" type="fixed">
         <parent link ="base_link"/>
-        <child link="shoulder_link"/>
+        <child link="shoulder_base"/>
         <origin xyz="0 0 1"/>
     </joint>
     <!-- SHOULDER -->
-    <link name = "shoulder_link">
-        <visual>
-            <origin xyz="0 0 -0.05"/>
+    <link name = "shoulder_base">
+        <!-- <visual>
+            <origin xyz="0 0 -0.5"/>
             <geometry>
-                <box size="0.1 0.1 0.1"/>
+                <box size="0.01 0.01 1"/>
             </geometry>
             <material name="blue"/>
-        </visual>
+        </visual> -->
     </link>
-    <joint name="shoulder_joint" type="revolute">
-        <parent link ="shoulder_link"/>
-        <child link="bicept_link"/>
-        <origin xyz="0 0 -0.1" rpy="0 0 0"/>
-        <axis xyz="0 1 0" rpy="0 0 0"/>
-        <limit lower="0" upper="${pi/2}" velocity ="100" effort = "100"/>
+   <joint name="shoulder_joint" type="revolute">
+        <origin xyz="0 0 0" rpy="${pi/2} 0 0"/>
+        <parent link ="shoulder_base"/>
+        <child link="shoulder_link"/>
+        <axis xyz="0 0 1" />
+        <limit lower="${-pi/2}" upper="${pi/4}" velocity ="100" effort = "100"/>
     </joint>
-    <link name = "bicept_link">
-        <visual>
+    <link name = "shoulder_link">
+        <!-- <visual>
             <origin xyz="0 0 0.5"/>
             <geometry>
@@ -45,15 +45,20 @@
             </geometry>
             <material name="orange"/>
-        </visual>
+        </visual> -->
     </link>
     <joint name="bicept_joint" type="revolute">
+        <parent link ="shoulder_link"/>
+        <child link="bicept_link"/>
+        <origin xyz="0.1 0 0" rpy="0 ${pi/2} 0"/>
+        <axis xyz="0 0 1" />
+        <limit lower="${-pi/2}" upper="${pi/2}" velocity ="100" effort = "100"/>
+    </joint>
+    <!-- <joint name="bicept_joint" type="fixed">
         <parent link ="bicept_link"/>
         <child link="elbow_link"/>
-        <origin xyz="0 0 0.1" rpy="0 0 0"/>
-        <axis xyz="0 1 0" rpy="0 0 0"/>
-        <limit lower="0" upper="${pi/2}" velocity ="100" effort = "100"/>
-    </joint>
-    <link name = "elbow_link">
-        <visual>
+        <origin xyz="0 0.5 0"/>
+    </joint>  -->
+    <link name = "bicept_link">
+        <!-- <visual>
             <origin xyz="0 0 0.05"/>
             <geometry>
@@ -61,5 +66,83 @@
             </geometry>
             <material name="white"/>
-        </visual>
+        </visual> -->
+    </link>
+    <joint name="elbow_joint" type="revolute">
+        <parent link ="bicept_link"/>
+        <child link="elbow_link"/>
+        <origin xyz="0 0 0.293" rpy="0 ${-pi/2} 0"/>
+        <axis xyz="0 0 1" />
+        <limit lower="0" upper="2.3562" velocity ="100" effort = "100"/>
+    </joint>
+    <link name = "elbow_link">
+        <!-- <visual>
+            <origin xyz="0 0 0.05"/>
+            <geometry>
+                <box size="0.1 0.11 0.1"/>
+            </geometry>
+            <material name="white"/>
+        </visual> -->
+    </link>
+    <joint name="forearm_joint" type="revolute">
+        <parent link ="elbow_link"/>
+        <child link="forearm_link"/>
+        <origin xyz="0.1 0 0" rpy="0 ${pi/2} 0"/>
+        <axis xyz="0 0 1" />
+        <limit lower="${-pi/2}" upper="${pi/2}" velocity ="100" effort = "100"/>
+    </joint>
+    <link name = "forearm_link">
+        <!-- <visual>
+            <origin xyz="0 0 0.05"/>
+            <geometry>
+                <box size="0.1 0.11 0.1"/>
+            </geometry>
+            <material name="white"/>
+        </visual> -->
+    </link>
+    <joint name="wrist_joint1" type="revolute">
+        <parent link ="forearm_link"/>
+        <child link="wrist_link1"/>
+        <origin xyz="0 0 0.2" rpy="${-pi/2} 0 0"/>
+        <axis xyz="0 0 1" />
+        <limit lower="${-pi/2}" upper="${pi/2}" velocity ="100" effort = "100"/>
+    </joint>
+    <link name = "wrist_link1">
+        <!-- <visual>
+            <origin xyz="0 0 0.05"/>
+            <geometry>
+                <box size="0.1 0.11 0.1"/>
+            </geometry>
+            <material name="white"/>
+        </visual> -->
+    </link>
+    <joint name="wrist_joint2" type="revolute">
+        <parent link ="wrist_link1"/>
+        <child link="wrist_link2"/>
+        <origin xyz="0 0 0" rpy="0 ${-pi/2} 0"/>
+        <axis xyz="0 0 1" />
+        <limit lower="${-pi/2}" upper="${pi/2}" velocity ="100" effort = "100"/>
+    </joint>
+    <link name = "wrist_link2">
+        <!-- <visual>
+            <origin xyz="0 0 0.05"/>
+            <geometry>
+                <box size="0.1 0.11 0.1"/>
+            </geometry>
+            <material name="white"/>
+        </visual> -->
+    </link>
+    <joint name="tip_joint" type="fixed">
+        <parent link ="wrist_link2"/>
+        <child link="tip"/>
+        <origin xyz="0 -1 0"/>
+    </joint>
+    <link name = "tip">
+        <!-- <visual>
+            <origin xyz="0 0 0.05"/>
+            <geometry>
+                <box size="0.1 0.11 0.1"/>
+            </geometry>
+            <material name="white"/>
+        </visual> -->
     </link>
 </robot>

Commit message: Installed odrive package

File: src/arm_urdf/description/robot_core.xacro (robot description, xacro)
@@ -15,4 +15,11 @@
     <!-- BASE -->
     <link name="base_link">
+        <visual>
+            <origin xyz="0 0 0.5"/>
+            <geometry>
+                <box size="0.05 0.05 1"/>
+            </geometry>
+            <material name="blue"/>
+        </visual>
     </link>
     <joint name="base_joint" type="fixed">
@@ -23,11 +30,4 @@
     <!-- SHOULDER -->
     <link name = "shoulder_base">
-        <!-- <visual>
-            <origin xyz="0 0 -0.5"/>
-            <geometry>
-                <box size="0.01 0.01 1"/>
-            </geometry>
-            <material name="blue"/>
-        </visual> -->
     </link>
    <joint name="shoulder_joint" type="revolute">
@@ -39,11 +39,11 @@
     </joint>
     <link name = "shoulder_link">
-        <!-- <visual>
-            <origin xyz="0 0 0.5"/>
+        <visual>
+            <origin xyz="0.05 0 0"/>
             <geometry>
-                <box size="0.01 0.01 0.1"/>
+                <box size="0.1 0.05 0.05"/>
             </geometry>
-            <material name="orange"/>
-        </visual> -->
+            <material name="white"/>
+        </visual>
     </link>
     <joint name="bicept_joint" type="revolute">
@@ -54,17 +54,12 @@
         <limit lower="${-pi/2}" upper="${pi/2}" velocity ="100" effort = "100"/>
     </joint>
-    <!-- <joint name="bicept_joint" type="fixed">
-        <parent link ="bicept_link"/>
-        <child link="elbow_link"/>
-        <origin xyz="0 0.5 0"/>
-    </joint>  -->
     <link name = "bicept_link">
-        <!-- <visual>
-            <origin xyz="0 0 0.05"/>
+        <visual>
+            <origin xyz="0 0 0.1465"/>
             <geometry>
-                <box size="0.1 0.11 0.1"/>
+                <box size="0.05 0.05 0.293"/>
             </geometry>
-            <material name="white"/>
-        </visual> -->
+            <material name="orange"/>
+        </visual>
     </link>
     <joint name="elbow_joint" type="revolute">
@@ -76,11 +71,11 @@
     </joint>
     <link name = "elbow_link">
-        <!-- <visual>
-            <origin xyz="0 0 0.05"/>
+        <visual>
+            <origin xyz="0.05 0 0"/>
             <geometry>
-                <box size="0.1 0.11 0.1"/>
+                <box size="0.1 0.05 0.05"/>
             </geometry>
-            <material name="white"/>
-        </visual> -->
+            <material name="blue"/>
+        </visual>
     </link>
     <joint name="forearm_joint" type="revolute">
@@ -92,11 +87,11 @@
     </joint>
     <link name = "forearm_link">
-        <!-- <visual>
-            <origin xyz="0 0 0.05"/>
+        <visual>
+            <origin xyz="0 0 0.1"/>
             <geometry>
-                <box size="0.1 0.11 0.1"/>
+                <box size="0.05 0.05 0.2"/>
             </geometry>
             <material name="white"/>
-        </visual> -->
+        </visual>
     </link>
     <joint name="wrist_joint1" type="revolute">
@@ -124,11 +119,11 @@
     </joint>
     <link name = "wrist_link2">
-        <!-- <visual>
-            <origin xyz="0 0 0.05"/>
+        <visual>
+            <origin xyz="0 -0.5 0"/>
             <geometry>
-                <box size="0.1 0.11 0.1"/>
+                <box size="0.02 1 0.02"/>
             </geometry>
-            <material name="white"/>
-        </visual> -->
+            <material name="orange"/>
+        </visual>
     </link>
     <joint name="tip_joint" type="fixed">
@@ -138,11 +133,11 @@
     </joint>
     <link name = "tip">
-        <!-- <visual>
-            <origin xyz="0 0 0.05"/>
+        <visual>
+            <origin xyz="0 0 0"/>
             <geometry>
-                <box size="0.1 0.11 0.1"/>
+                <box size="0.1 0.1 0.1"/>
             </geometry>
             <material name="white"/>
-        </visual> -->
+        </visual>
     </link>
 <!-- Hello hello even more hellos-->

Commit message: added collisiion and inertia tags. rogot doesnt show up on gazebo

File: src/arm_urdf/description/robot_core.xacro (robot description, xacro)
@@ -1,4 +1,5 @@
 <?xml version="1.0"?>
 <robot xmlns:xacro="http://www.ros.org/wiki/xacro" >
+    <xacro:include filename="inertial_macros.xacro"/>
     <material name="white">
         <color rgba="1 1 1 1"/>
@@ -22,4 +23,10 @@
             <material name="blue"/>
         </visual>
+        <collision>
+            <origin xyz="0 0 0.5"/>
+            <geometry>
+                <box size="0.05 0.05 1"/>
+            </geometry>
+        </collision>
     </link>
     <joint name="base_joint" type="fixed">
@@ -46,4 +53,13 @@
             <material name="white"/>
         </visual>
+        <collision>
+            <origin xyz="0.05 0 0"/>
+            <geometry>
+                <box size="0.1 0.05 0.05"/>
+            </geometry>
+        </collision>
+        <xacro:inertial_box mass="0.5" x="0.1" y="0.05" z="0.05">
+            <origin xyz="0.05 0 0" rpy= "0 0 0"/>
+        </xacro:inertial_box >
     </link>
     <joint name="bicept_joint" type="revolute">
@@ -62,4 +78,13 @@
             <material name="orange"/>
         </visual>
+        <collision>
+            <origin xyz="0 0 0.1465"/>
+            <geometry>
+                <box size="0.05 0.05 0.293"/>
+            </geometry>
+        </collision>
+        <xacro:inertial_box mass = "3" x="0.05" y="0.05" z="0.293">
+            <origin xyz="0 0 0.1465" rpy= "0 0 0"/>
+        </xacro:inertial_box >
     </link>
     <joint name="elbow_joint" type="revolute">
@@ -78,4 +103,13 @@
             <material name="blue"/>
         </visual>
+        <collision>
+            <origin xyz="0.05 0 0"/>
+            <geometry>
+                <box size="0.1 0.05 0.05"/>
+            </geometry>
+        </collision>
+        <xacro:inertial_box mass ="0.6" x="0.1" y="0.05" z="0.05">
+            <origin xyz="0.05 0 0" rpy= "0 0 0"/>
+        </xacro:inertial_box >
     </link>
     <joint name="forearm_joint" type="revolute">
@@ -94,4 +128,13 @@
             <material name="white"/>
         </visual>
+        <collision>
+            <origin xyz="0 0 0.1"/>
+            <geometry>
+                <box size="0.05 0.05 0.2"/>
+            </geometry>
+        </collision>
+        <xacro:inertial_box mass ="2.5" x="0.05" y="0.05" z="0.2">
+            <origin xyz="0 0 0.1" rpy= "0 0 0"/>
+        </xacro:inertial_box >
     </link>
     <joint name="wrist_joint1" type="revolute">
@@ -103,11 +146,4 @@
     </joint>
     <link name = "wrist_link1">
-        <!-- <visual>
-            <origin xyz="0 0 0.05"/>
-            <geometry>
-                <box size="0.1 0.11 0.1"/>
-            </geometry>
-            <material name="white"/>
-        </visual> -->
     </link>
     <joint name="wrist_joint2" type="revolute">
@@ -126,4 +162,13 @@
             <material name="orange"/>
         </visual>
+        <collision>
+            <origin xyz="0 -0.5 0"/>
+            <geometry>
+                <box size="0.02 1 0.02"/>
+            </geometry>
+        </collision>
+        <xacro:inertial_box mass ="0.5" x="0.2" y="1" z="0.2">
+            <origin xyz="0 -0.5 0" rpy= "0 0 0"/>
+        </xacro:inertial_box >
     </link>
     <joint name="tip_joint" type="fixed">
@@ -136,8 +181,14 @@
             <origin xyz="0 0 0"/>
             <geometry>
-                <box size="0.1 0.1 0.1"/>
+                <box size="0.05 0.05 0.05"/>
             </geometry>
             <material name="white"/>
         </visual>
+        <collision>
+            <origin xyz="0 0 0"/>
+            <geometry>
+                <box size="0.05 0.05 0.05"/>
+            </geometry>
+        </collision>
     </link>
 <!-- Hello hello even more hellos-->

Commit message: Added STl meshes, currently orienting

File: src/arm_urdf/description/robot_core.xacro (robot description, xacro)
@@ -17,24 +17,32 @@
     <link name="base_link">
         <visual>
+            <origin xyz="-0.6052 -0.31115 0"/>
+            <geometry>
+                <mesh filename="package://arm_urdf/meshes/base.stl" scale="0.001 0.001 0.001 "/>
+            </geometry>
+            <material name="white"/>
+        </visual>
+        <collision>
             <origin xyz="0 0 0.5"/>
             <geometry>
                 <box size="0.05 0.05 1"/>
             </geometry>
-            <material name="blue"/>
-        </visual>
-        <collision>
-            <origin xyz="0 0 0.5"/>
-            <geometry>
-                <box size="0.05 0.05 1"/>
-            </geometry>
-        </collision>
-    </link>
+        </collision>
+    </link>
+    <!-- SETS THE HEIGHT OF THE ARM -->
     <joint name="base_joint" type="fixed">
         <parent link ="base_link"/>
         <child link="shoulder_base"/>
-        <origin xyz="0 0 1"/>
+        <origin xyz="0 0 1.175"/>
     </joint>
     <!-- SHOULDER -->
     <link name = "shoulder_base">
+        <visual>
+            <origin xyz="-0.0425 -0.09775 -0.05"/>
+            <geometry>
+                <mesh filename="package://arm_urdf/meshes/shoulder_base.stl" scale="0.001 0.001 0.001 "/>
+            </geometry>
+            <material name="white"/>
+        </visual>
     </link>
    <joint name="shoulder_joint" type="revolute">
@@ -47,14 +55,14 @@
     <link name = "shoulder_link">
         <visual>
+            <origin xyz="0 -0.075 0.075" rpy ="0 ${pi/2} 0"/>
+            <geometry>
+                <mesh filename="package://arm_urdf/meshes/shoulder.stl" scale="0.001 0.001 0.001 "/>
+            </geometry>
+            <material name="white"/>
+        </visual>
+        <collision>
             <origin xyz="0.05 0 0"/>
             <geometry>
-                <box size="0.1 0.05 0.05"/>
-            </geometry>
-            <material name="white"/>
-        </visual>
-        <collision>
-            <origin xyz="0.05 0 0"/>
-            <geometry>
-                <box size="0.1 0.05 0.05"/>
+                <mesh filename="package://arm_urdf/meshes/shoulder.stl" scale="0.001 0.001 0.001 "/>
             </geometry>
         </collision>
@@ -66,5 +74,5 @@
         <parent link ="shoulder_link"/>
         <child link="bicept_link"/>
-        <origin xyz="0.1 0 0" rpy="0 ${pi/2} 0"/>
+        <origin xyz="0.125 0 0" rpy="0 ${pi/2} 0"/>
         <axis xyz="0 0 1" />
         <limit lower="${-pi/2}" upper="${pi/2}" velocity ="100" effort = "100"/>
@@ -72,14 +80,14 @@
     <link name = "bicept_link">
         <visual>
+            <origin xyz="0 0 0.35" rpy="0 ${pi/2} 0"/>
+            <geometry>
+                <mesh filename="package://arm_urdf/meshes/bicept.stl" scale="0.001 0.001 0.001 "/>
+            </geometry>
+            <material name="orange"/>
+        </visual>
+        <collision>
             <origin xyz="0 0 0.1465"/>
             <geometry>
-                <box size="0.05 0.05 0.293"/>
-            </geometry>
-            <material name="orange"/>
-        </visual>
-        <collision>
-            <origin xyz="0 0 0.1465"/>
-            <geometry>
-                <box size="0.05 0.05 0.293"/>
+                <mesh filename="package://arm_urdf/meshes/bicept.stl" scale="0.001 0.001 0.001 "/>
             </geometry>
         </collision>
@@ -99,5 +107,5 @@
             <origin xyz="0.05 0 0"/>
             <geometry>
-                <box size="0.1 0.05 0.05"/>
+                <mesh filename="package://arm_urdf/meshes/elbow.stl" scale="0.001 0.001 0.001 "/>
             </geometry>
             <material name="blue"/>
@@ -106,5 +114,5 @@
             <origin xyz="0.05 0 0"/>
             <geometry>
-                <box size="0.1 0.05 0.05"/>
+                <mesh filename="package://arm_urdf/meshes/elbow.stl" scale="0.001 0.001 0.001 "/>
             </geometry>
         </collision>
@@ -124,5 +132,5 @@
             <origin xyz="0 0 0.1"/>
             <geometry>
-                <box size="0.05 0.05 0.2"/>
+                <mesh filename="package://arm_urdf/meshes/forearm.stl" scale="0.001 0.001 0.001 "/>
             </geometry>
             <material name="white"/>
@@ -131,5 +139,5 @@
             <origin xyz="0 0 0.1"/>
             <geometry>
-                <box size="0.05 0.05 0.2"/>
+                <mesh filename="package://arm_urdf/meshes/forearm.stl" scale="0.001 0.001 0.001 "/>
             </geometry>
         </collision>
@@ -146,4 +154,11 @@
     </joint>
     <link name = "wrist_link1">
+        <visual>
+            <origin xyz="0 0 0.1"/>
+            <geometry>
+                <mesh filename="package://arm_urdf/meshes/wrist_1.stl" scale="0.001 0.001 0.001 "/>
+            </geometry>
+            <material name="white"/>
+        </visual>
     </link>
     <joint name="wrist_joint2" type="revolute">
@@ -158,5 +173,5 @@
             <origin xyz="0 -0.5 0"/>
             <geometry>
-                <box size="0.02 1 0.02"/>
+                <mesh filename="package://arm_urdf/meshes/wrist_2.stl" scale="0.001 0.001 0.001 "/>
             </geometry>
             <material name="orange"/>
@@ -165,5 +180,5 @@
             <origin xyz="0 -0.5 0"/>
             <geometry>
-                <box size="0.02 1 0.02"/>
+                <mesh filename="package://arm_urdf/meshes/wrist_2.stl" scale="0.001 0.001 0.001 "/>
             </geometry>
         </collision>
@@ -192,4 +207,3 @@
         </collision>
     </link>
-<!-- Hello hello even more hellos-->
 </robot>
