Commit message: finished visual UDRF params

File: src/arm_urdf/description/robot_core.xacro (robot description, xacro)
@@ -43,5 +43,5 @@
                 <mesh filename="package://arm_urdf/meshes/shoulder_base.stl" scale="0.001 0.001 0.001 "/>
             </geometry>
-            <material name="white"/>
+            <material name="black"/>
         </visual>
     </link>
@@ -51,13 +51,13 @@
         <child link="shoulder_link"/>
         <axis xyz="0 0 1" />
-        <limit lower="${-pi/2}" upper="${pi/4}" velocity ="100" effort = "100"/>
+        <limit lower="${-pi/2}" upper="0.4" velocity ="100" effort = "100"/>
     </joint>
     <link name = "shoulder_link">
         <visual>
-            <origin xyz="0 -0.075 0.075" rpy ="0 ${pi/2} 0"/>
+            <origin xyz="-0.05 -0.075 0.075" rpy ="0 ${pi/2} 0"/>
             <geometry>
                 <mesh filename="package://arm_urdf/meshes/shoulder.stl" scale="0.001 0.001 0.001 "/>
             </geometry>
-            <material name="white"/>
+            <material name="blue"/>
         </visual>
         <collision>
@@ -74,5 +74,5 @@
         <parent link ="shoulder_link"/>
         <child link="bicept_link"/>
-        <origin xyz="0.125 0 0" rpy="0 ${pi/2} 0"/>
+        <origin xyz="0.05 0 0" rpy="0 ${pi/2} 0"/>
         <axis xyz="0 0 1" />
         <limit lower="${-pi/2}" upper="${pi/2}" velocity ="100" effort = "100"/>
@@ -80,5 +80,5 @@
     <link name = "bicept_link">
         <visual>
-            <origin xyz="0 0 0.35" rpy="0 ${pi/2} 0"/>
+            <origin xyz="0.050 -0.060 0.383" rpy="0 ${pi/2} ${pi/2}"/>
             <geometry>
                 <mesh filename="package://arm_urdf/meshes/bicept.stl" scale="0.001 0.001 0.001 "/>
@@ -99,11 +99,11 @@
         <parent link ="bicept_link"/>
         <child link="elbow_link"/>
-        <origin xyz="0 0 0.293" rpy="0 ${-pi/2} 0"/>
-        <axis xyz="0 0 1" />
-        <limit lower="0" upper="2.3562" velocity ="100" effort = "100"/>
+        <origin xyz="0 0 0.343" rpy="0 ${-pi/2} 0"/>
+        <axis xyz="0 0 1" />
+        <limit lower="0" upper="2" velocity ="100" effort = "100"/>
     </joint>
     <link name = "elbow_link">
         <visual>
-            <origin xyz="0.05 0 0"/>
+            <origin xyz="0.049 -0.04 -0.0286" rpy ="0 0 ${pi/2}"/>
             <geometry>
                 <mesh filename="package://arm_urdf/meshes/elbow.stl" scale="0.001 0.001 0.001 "/>
@@ -124,5 +124,5 @@
         <parent link ="elbow_link"/>
         <child link="forearm_link"/>
-        <origin xyz="0.1 0 0" rpy="0 ${pi/2} 0"/>
+        <origin xyz="0.038 0 0" rpy="0 ${pi/2} 0"/>
         <axis xyz="0 0 1" />
         <limit lower="${-pi/2}" upper="${pi/2}" velocity ="100" effort = "100"/>
@@ -130,9 +130,9 @@
     <link name = "forearm_link">
         <visual>
-            <origin xyz="0 0 0.1"/>
+            <origin xyz="0.042 -0.04 0.289" rpy ="0 ${pi/2} ${pi/2}"/>
             <geometry>
                 <mesh filename="package://arm_urdf/meshes/forearm.stl" scale="0.001 0.001 0.001 "/>
             </geometry>
-            <material name="white"/>
+            <material name="orange"/>
         </visual>
         <collision>
@@ -149,15 +149,15 @@
         <parent link ="forearm_link"/>
         <child link="wrist_link1"/>
-        <origin xyz="0 0 0.2" rpy="${-pi/2} 0 0"/>
-        <axis xyz="0 0 1" />
-        <limit lower="${-pi/2}" upper="${pi/2}" velocity ="100" effort = "100"/>
+        <origin xyz="0 0 0.264" rpy="${-pi/2} 0 0"/>
+        <axis xyz="1 0 0" />
+        <limit lower="-0.3" upper="1" velocity ="100" effort = "100"/>
     </joint>
     <link name = "wrist_link1">
         <visual>
-            <origin xyz="0 0 0.1"/>
+            <origin xyz="-0.05 -0.025 -0.02502" rpy="0 ${-pi/2} ${-pi/2} " />
             <geometry>
                 <mesh filename="package://arm_urdf/meshes/wrist_1.stl" scale="0.001 0.001 0.001 "/>
             </geometry>
-            <material name="white"/>
+            <material name="blue"/>
         </visual>
     </link>
@@ -166,10 +166,10 @@
         <child link="wrist_link2"/>
         <origin xyz="0 0 0" rpy="0 ${-pi/2} 0"/>
-        <axis xyz="0 0 1" />
-        <limit lower="${-pi/2}" upper="${pi/2}" velocity ="100" effort = "100"/>
+        <axis xyz="1 0 0" />
+        <limit lower="${-pi/4}" upper="${pi/4}" velocity ="100" effort = "100"/>
     </joint>
     <link name = "wrist_link2">
         <visual>
-            <origin xyz="0 -0.5 0"/>
+            <origin xyz="0.0435 -0.0235 -0.0235" rpy="${-pi/2} ${-pi} 0"/>
             <geometry>
                 <mesh filename="package://arm_urdf/meshes/wrist_2.stl" scale="0.001 0.001 0.001 "/>
@@ -190,19 +190,28 @@
         <parent link ="wrist_link2"/>
         <child link="tip"/>
-        <origin xyz="0 -1 0"/>
+        <origin xyz="0 -0.9 0"/>
     </joint>
     <link name = "tip">
+        <!-- SQUARE TIP -->
         <visual>
             <origin xyz="0 0 0"/>
             <geometry>
+                <box size="0.025 0.025 0.025"/>
+            </geometry>
+            <material name="white"/>
+        </visual>
+        <!-- BLADE -->
+        <visual>
+            <origin xyz="0 0.45 0"/>
+            <geometry>
+                <box size="0.01 0.9 0.01" length="1"/>
+            </geometry>
+            <material name="white"/>
+        </visual>
+        <collision>
+            <origin xyz="0 0 0"/>
+            <geometry>
                 <box size="0.05 0.05 0.05"/>
             </geometry>
-            <material name="white"/>
-        </visual>
-        <collision>
-            <origin xyz="0 0 0"/>
-            <geometry>
-                <box size="0.05 0.05 0.05"/>
-            </geometry>
         </collision>
     </link>
