Commit message: Added collision properties and terminal_commands.txt

File: src/arm_urdf/description/gazebo_control.xacro (robot description, xacro)
@@ -2,14 +2,41 @@
 <robot xmlns:xacro="http://www.ros.org/wiki/xacro">
     <gazebo>
+        <gazebo reference= "base_link">
+            <material>Gazebo/White</material>
+        </gazebo>
+        <gazebo reference= "shoulder_base">
+            <material>Gazebo/Black</material>
+        </gazebo>
+        <gazebo reference= "shoulder_link">
+            <material>Gazebo/Orange</material>
+        </gazebo>
+        <gazebo reference= "elbow_link">
+            <material>Gazebo/Blue</material>
+        </gazebo>
+        <gazebo reference= "forearm_link">
+            <material>Gazebo/Orange</material>
+        </gazebo>
+        <gazebo reference= "wrist_link1">
+            <material>Gazebo/Blue</material>
+        </gazebo>
+        <gazebo reference= "wrist_link2">
+            <material>Gazebo/Orange</material>
+        </gazebo>
+        <gazebo reference= "tip">
+            <material>Gazebo/White</material>
+        </gazebo>
+    </gazebo>
+</robot>
+    <!-- <gazebo>
         <plugin name="diff_drive" filename="libgazebo_ros_diff_drive.so">
-            <!-- Wheel Information -->
+            Wheel Information
             <left_joint>left_wheel_joint</left_joint>
             <right_joint>right_wheel_joint</right_joint>
             <wheel_separation>0.297</wheel_separation>
             <wheel_diameter>0.066</wheel_diameter>
-            <!-- Limits -->
+            Limits
             <max_wheel_torque>200</max_wheel_torque>
             <max_wheel_acceleration>10.0</max_wheel_acceleration>
-            <!-- Output -->
+            Output
             <odometry_frame>odom</odometry_frame>
             <robot_base_frame>base_link</robot_base_frame>
@@ -18,4 +45,3 @@
             <publish_wheel_tf>true</publish_wheel_tf>
         </plugin>
-    </gazebo>
-</robot>
+    </gazebo> -->

File: src/arm_urdf/description/robot_core.xacro (robot description, xacro)
@@ -24,7 +24,7 @@
         </visual>
         <collision>
-            <origin xyz="0 0 0.5"/>
-            <geometry>
-                <box size="0.05 0.05 1"/>
+            <origin xyz="-0.6052 -0.31115 0"/>
+            <geometry>
+                <mesh filename="package://arm_urdf/meshes/base.stl" scale="0.001 0.001 0.001 "/>
             </geometry>
         </collision>
@@ -45,4 +45,10 @@
             <material name="black"/>
         </visual>
+        <collision>
+            <origin xyz="-0.0425 -0.09775 -0.05"/>
+            <geometry>
+                <mesh filename="package://arm_urdf/meshes/shoulder_base.stl" scale="0.001 0.001 0.001 "/>
+            </geometry>
+        </collision>
     </link>
    <joint name="shoulder_joint" type="revolute">
@@ -62,5 +68,5 @@
         </visual>
         <collision>
-            <origin xyz="0.05 0 0"/>
+            <origin xyz="-0.05 -0.075 0.075" rpy ="0 ${pi/2} 0"/>
             <geometry>
                 <mesh filename="package://arm_urdf/meshes/shoulder.stl" scale="0.001 0.001 0.001 "/>
@@ -87,5 +93,5 @@
         </visual>
         <collision>
-            <origin xyz="0 0 0.1465"/>
+            <origin xyz="0.050 -0.060 0.383" rpy="0 ${pi/2} ${pi/2}"/>
             <geometry>
                 <mesh filename="package://arm_urdf/meshes/bicept.stl" scale="0.001 0.001 0.001 "/>
@@ -112,5 +118,5 @@
         </visual>
         <collision>
-            <origin xyz="0.05 0 0"/>
+            <origin xyz="0.049 -0.04 -0.0286" rpy ="0 0 ${pi/2}"/>
             <geometry>
                 <mesh filename="package://arm_urdf/meshes/elbow.stl" scale="0.001 0.001 0.001 "/>
@@ -137,5 +143,5 @@
         </visual>
         <collision>
-            <origin xyz="0 0 0.1"/>
+            <origin xyz="0.042 -0.04 0.289" rpy ="0 ${pi/2} ${pi/2}"/>
             <geometry>
                 <mesh filename="package://arm_urdf/meshes/forearm.stl" scale="0.001 0.001 0.001 "/>
@@ -161,4 +167,10 @@
             <material name="blue"/>
         </visual>
+        <collision>
+            <origin xyz="-0.05 -0.025 -0.02502" rpy="0 ${-pi/2} ${-pi/2} " />
+            <geometry>
+                <mesh filename="package://arm_urdf/meshes/wrist_1.stl" scale="0.001 0.001 0.001 "/>
+            </geometry>
+        </collision>
     </link>
     <joint name="wrist_joint2" type="revolute">
@@ -178,5 +190,5 @@
         </visual>
         <collision>
-            <origin xyz="0 -0.5 0"/>
+            <origin xyz="0.0435 -0.0235 -0.0235" rpy="${-pi/2} ${-pi} 0"/>
             <geometry>
                 <mesh filename="package://arm_urdf/meshes/wrist_2.stl" scale="0.001 0.001 0.001 "/>
@@ -216,3 +228,4 @@
         </collision>
     </link>
+    <xacro:include filename= "gazebo_control.xacro"/>
 </robot>
