Commit message: 1st version of ros2 control and moveit config

File: src/arm_urdf/description/arm.urdf (robot description, URDF)
Before this commit: robot arm, 9 links, 8 joints
Links:
- link base_link: mass 2.5 -> 40
- link bicept_link: mass 3 -> 2.2
- link elbow_link: mass 0.6 -> 0.5
- link forearm_link: mass 2.5 -> 1.5
- link shoulder_base: mass 2.5 -> 1
- link shoulder_link: mass 0.5 -> 1
- link tip: mass 2.5 -> 0.5; geometry collision box size=0.01 0.9 0.01; collision box size=0.025 0.025 0.025
- link wrist_link1: mass 2.5 -> 0.5
- link wrist_link2: mass 0.5 -> 0.2

File: src/arm_urdf/description/gazebo_control.xacro (robot description, xacro)
@@ -2,28 +2,4 @@
 <robot xmlns:xacro="http://www.ros.org/wiki/xacro">
     <gazebo>
-        <gazebo reference= "base_link">
-            <material>Gazebo/White</material>
-        </gazebo>
-        <gazebo reference= "shoulder_base">
-            <material>Gazebo/Black</material>
-        </gazebo>
-        <gazebo reference= "shoulder_link">
-            <material>Gazebo/Orange</material>
-        </gazebo>
-        <gazebo reference= "elbow_link">
-            <material>Gazebo/Blue</material>
-        </gazebo>
-        <gazebo reference= "forearm_link">
-            <material>Gazebo/Orange</material>
-        </gazebo>
-        <gazebo reference= "wrist_link1">
-            <material>Gazebo/Blue</material>
-        </gazebo>
-        <gazebo reference= "wrist_link2">
-            <material>Gazebo/Orange</material>
-        </gazebo>
-        <gazebo reference= "tip">
-            <material>Gazebo/White</material>
-        </gazebo>
     </gazebo>
 </robot>

File: src/arm_urdf/description/robot.urdf.xacro (robot description, xacro)
@@ -2,4 +2,5 @@
 <robot xmlns:xacro="http://www.ros.org/wiki/xacro"  name="robot">
     <xacro:include filename= "robot_core.xacro"/>
-    <xacro:include filename= "gazebo_control.xacro"/>
+    <!-- <xacro:include filename= "gazebo_control.xacro"/> -->
+    <xacro:include filename= "ros2_control.xacro"/>
 </robot>

File: src/arm_urdf/description/ros2_control.xacro (robot description, xacro)
@@ -1,5 +1,5 @@
 <?xml version="1.0"?>
 <robot xmlns:xacro="http://www.ros.org/wiki/xacro">
-    <xacro:unless value="$(arg sim_mode)">
+    <!-- <xacro:unless value="$(arg sim_mode)">
         <ros2_control name="RealRobot" type="system">
             <hardware>
@@ -30,32 +30,85 @@
             </joint>
         </ros2_control>
-    </xacro:unless>
-    <xacro:if value="$(arg sim_mode)">
+    </xacro:unless> -->
+    <!-- <joint name="shoulder_joint">
+        <command_interface name="position"/>
+        <state_interface name="position">
+          <param name="initial_value">${initial_positions['shoulder_joint']}</param>
+        </state_interface>
+        <state_interface name="velocity"/>
+    </joint>
+    <joint name="bicept_joint">
+        <command_interface name="position"/>
+        <state_interface name="position">
+          <param name="initial_value">${initial_positions['bicept_joint']}</param>
+        </state_interface>
+        <state_interface name="velocity"/>
+    </joint> -->
+    <!-- <xacro:if value="$(arg sim_mode)"> -->
         <ros2_control name="GazeboSystem" type="system">
             <hardware>
                 <plugin>gazebo_ros2_control/GazeboSystem</plugin>
             </hardware>
-            <joint name="left_wheel_joint">
-                <command_interface name="velocity">
-                    <param name="min">-10</param>
-                    <param name="max">10</param>
+            <joint name="shoulder_joint">
+                <command_interface name="position">
+                    <param name="min">-1</param>
+                    <param name="max">1</param>
                 </command_interface>
+                <state_interface name="effort"/>
                 <state_interface name="velocity"/>
                 <state_interface name="position"/>
             </joint>
-            <joint name="right_wheel_joint">
-                <command_interface name="velocity">
-                    <param name="min">-10</param>
-                    <param name="max">10</param>
+            <joint name="bicept_joint">
+                <command_interface name="position">
+                    <param name="min">-1</param>
+                    <param name="max">1</param>
                 </command_interface>
+                <state_interface name="effort"/>
+                <state_interface name="velocity"/>
+                <state_interface name="position"/>
+            </joint>
+            <joint name="elbow_joint">
+                <command_interface name="position">
+                    <param name="min">-1</param>
+                    <param name="max">1</param>
+                </command_interface>
+                <state_interface name="effort"/>
+                <state_interface name="velocity"/>
+                <state_interface name="position"/>
+            </joint>
+            <joint name="forearm_joint">
+                <command_interface name="position">
+                    <param name="min">-1</param>
+                    <param name="max">1</param>
+                </command_interface>
+                <state_interface name="effort"/>
+                <state_interface name="velocity"/>
+                <state_interface name="position"/>
+            </joint>
+            <joint name="wrist_joint1">
+                <command_interface name="position">
+                    <param name="min">-1</param>
+                    <param name="max">1</param>
+                </command_interface>
+                <state_interface name="effort"/>
+                <state_interface name="velocity"/>
+                <state_interface name="position"/>
+            </joint>
+            <joint name="wrist_joint2">
+                <command_interface name="position">
+                    <param name="min">-1</param>
+                    <param name="max">1</param>
+                </command_interface>
+                <state_interface name="effort"/>
                 <state_interface name="velocity"/>
                 <state_interface name="position"/>
             </joint>
         </ros2_control>
-    </xacro:if>
+    <!-- </xacro:if> -->
     <gazebo>
         <plugin name="gazebo_ros2_control" filename="libgazebo_ros2_control.so">
+            <!-- Tells where to find controller information for Ros2 -->
             <parameters>$(find arm_urdf)/config/my_controllers.yaml</parameters>
-            <parameters>$(find arm_urdf)/config/gaz_ros2_ctl_use_sim.yaml</parameters>
+            <!-- <parameters>$(find arm_urdf)/config/gaz_ros2_ctl_use_sim.yaml</parameters> -->
         </plugin>
     </gazebo>
