Commit message: completed moveit motion planning

File: install/moveit_config/share/moveit_config/config/robot.ros2_control.xacro (robot description, xacro)
@@ -1,60 +1 @@
-<?xml version="1.0"?>
-<robot xmlns:xacro="http://www.ros.org/wiki/xacro">
-    <xacro:macro name="robot_ros2_control" params="name initial_positions_file">
-        <xacro:property name="initial_positions" value="${load_yaml(initial_positions_file)['initial_positions']}"/>
-        <ros2_control name="${name}" type="system">
-            <hardware>
-                <!-- By default, set up controllers for simulation. This won't work on real hardware -->
-                <plugin>mock_components/GenericSystem</plugin>
-            </hardware>
-            <joint name="shoulder_joint">
-                <command_interface name="position"/>
-                <state_interface name="position">
-                  <param name="initial_value">${initial_positions['shoulder_joint']}</param>
-                </state_interface>
-                <state_interface name="velocity"/>
-                <state_interface name="effort"/>
-            </joint>
-            <joint name="bicept_joint">
-                <command_interface name="position"/>
-                <state_interface name="position">
-                  <param name="initial_value">${initial_positions['bicept_joint']}</param>
-                </state_interface>
-                <state_interface name="velocity"/>
-                <state_interface name="effort"/>
-            </joint>
-            <joint name="elbow_joint">
-                <command_interface name="position"/>
-                <state_interface name="position">
-                  <param name="initial_value">${initial_positions['elbow_joint']}</param>
-                </state_interface>
-                <state_interface name="velocity"/>
-                <state_interface name="effort"/>
-            </joint>
-            <joint name="forearm_joint">
-                <command_interface name="position"/>
-                <state_interface name="position">
-                  <param name="initial_value">${initial_positions['forearm_joint']}</param>
-                </state_interface>
-                <state_interface name="velocity"/>
-                <state_interface name="effort"/>
-            </joint>
-            <joint name="wrist_joint1">
-                <command_interface name="position"/>
-                <state_interface name="position">
-                  <param name="initial_value">${initial_positions['wrist_joint1']}</param>
-                </state_interface>
-                <state_interface name="velocity"/>
-                <state_interface name="effort"/>
-            </joint>
-            <joint name="wrist_joint2">
-                <command_interface name="position"/>
-                <state_interface name="position">
-                  <param name="initial_value">${initial_positions['wrist_joint2']}</param>
-                </state_interface>
-                <state_interface name="velocity"/>
-                <state_interface name="effort"/>
-            </joint>
-        </ros2_control>
-    </xacro:macro>
-</robot>
+/home/jiaan/arm_project/src/moveit_config/config/robot.ros2_control.xacro

File: install/moveit_config/share/moveit_config/config/robot.urdf.xacro (robot description, xacro)
@@ -1,9 +1 @@
-<?xml version="1.0"?>
-<robot xmlns:xacro="http://www.ros.org/wiki/xacro" name="robot">
-    <xacro:arg name="initial_positions_file" default="initial_positions.yaml" />
-    <!-- Import robot urdf file -->
-    <xacro:include filename="$(find arm_urdf)/description/arm.urdf" />
-    <!-- Import control_xacro -->
-    <xacro:include filename="robot.ros2_control.xacro" />
-    <xacro:robot_ros2_control name="FakeSystem" initial_positions_file="$(arg initial_positions_file)"/>
-</robot>
+/home/jiaan/arm_project/src/moveit_config/config/robot.urdf.xacro

File: src/moveit_config/config/robot.ros2_control.xacro (robot description, xacro)
@@ -14,5 +14,4 @@
                 </state_interface>
                 <state_interface name="velocity"/>
-                <state_interface name="effort"/>
             </joint>
             <joint name="bicept_joint">
@@ -22,5 +21,4 @@
                 </state_interface>
                 <state_interface name="velocity"/>
-                <state_interface name="effort"/>
             </joint>
             <joint name="elbow_joint">
@@ -30,5 +28,4 @@
                 </state_interface>
                 <state_interface name="velocity"/>
-                <state_interface name="effort"/>
             </joint>
             <joint name="forearm_joint">
@@ -38,5 +35,4 @@
                 </state_interface>
                 <state_interface name="velocity"/>
-                <state_interface name="effort"/>
             </joint>
             <joint name="wrist_joint1">
@@ -46,5 +42,4 @@
                 </state_interface>
                 <state_interface name="velocity"/>
-                <state_interface name="effort"/>
             </joint>
             <joint name="wrist_joint2">
@@ -54,5 +49,4 @@
                 </state_interface>
                 <state_interface name="velocity"/>
-                <state_interface name="effort"/>
             </joint>
         </ros2_control>
