Commit message: updates to pi.launch.py

File: src/moveit_config/config/robot.ros2_control.xacro (robot description, xacro)
@@ -3,14 +3,26 @@
     <xacro:macro name="robot_ros2_control" params="name initial_positions_file">
         <xacro:property name="initial_positions" value="${load_yaml(initial_positions_file)['initial_positions']}"/>
+        <!-- CHANGE VALUE TO "false" IF USING REAL HARDWARE -->
+        <xacro:property name="use_sim" value="false"/>
         <ros2_control name="${name}" type="system">
+          <xacro:unless value="${use_sim}">
             <hardware>
-                <!-- By default, set up controllers for simulation. This won't work on real hardware -->
-                <plugin>gazebo_ros2_control/GazeboSystem</plugin>
-                <!-- <plugin>mock_components/GenericSystem</plugin> -->
+              <plugin>odrive_ros2_control_plugin/ODriveHardwareInterface</plugin>
+              <param name="can">can0</param>
             </hardware>
+          </xacro:unless>
+          <xacro:if value="${use_sim}">
+            <hardware>
+              <!-- By default, set up controllers for simulation. This won't work on real hardware -->
+              <plugin>gazebo_ros2_control/GazeboSystem</plugin>
+              <!-- <plugin>mock_components/GenericSystem</plugin> -->
+          </hardware>
+          </xacro:if>
+            <!-- JOINT DETAILS -->
             <joint name="shoulder_joint">
                 <command_interface name="position"/>
                 <state_interface name="position">
                   <param name="initial_value">${initial_positions['shoulder_joint']}</param>
+                  <param name="node_id">0</param>
                 </state_interface>
                 <state_interface name="velocity"/>
@@ -20,4 +32,5 @@
                 <state_interface name="position">
                   <param name="initial_value">${initial_positions['bicept_joint']}</param>
+                  <param name="node_id">1</param>
                 </state_interface>
                 <state_interface name="velocity"/>
@@ -27,4 +40,5 @@
                 <state_interface name="position">
                   <param name="initial_value">${initial_positions['elbow_joint']}</param>
+                  <param name="node_id">2</param>
                 </state_interface>
                 <state_interface name="velocity"/>
@@ -34,4 +48,5 @@
                 <state_interface name="position">
                   <param name="initial_value">${initial_positions['forearm_joint']}</param>
+                  <param name="node_id">3</param>
                 </state_interface>
                 <state_interface name="velocity"/>
@@ -41,4 +56,5 @@
                 <state_interface name="position">
                   <param name="initial_value">${initial_positions['wrist_joint1']}</param>
+                  <param name="node_id">4</param>
                 </state_interface>
                 <state_interface name="velocity"/>
@@ -48,8 +64,10 @@
                 <state_interface name="position">
                   <param name="initial_value">${initial_positions['wrist_joint2']}</param>
+                  <param name="node_id">5</param>
                 </state_interface>
                 <state_interface name="velocity"/>
             </joint>
         </ros2_control>
+        <!-- ONLY NEEDED FOR GAZEBO -->
         <gazebo>
           <plugin name="gazebo_ros2_control" filename="libgazebo_ros2_control.so">

Commit message: ros2 control on rasp pi

File: src/moveit_config/config/robot.ros2_control.xacro (robot description, xacro)
@@ -1,27 +1,22 @@
 <?xml version="1.0"?>
 <robot xmlns:xacro="http://www.ros.org/wiki/xacro">
-    <xacro:macro name="robot_ros2_control" params="name initial_positions_file">
-        <xacro:property name="initial_positions" value="${load_yaml(initial_positions_file)['initial_positions']}"/>
+    <!-- <xacro:macro name="robot_ros2_control" params="name initial_positions_file"> -->
+    <!-- <xacro:macro name="robot_ros2_control" params="name"> -->
+    <!-- <xacro:arg name="initial_positions_file" default="initial_positions.yaml" />
+        <xacro:property name="initial_positions" value="${load_yaml(initial_positions_file)['initial_positions']}"/> -->
         <!-- CHANGE VALUE TO "false" IF USING REAL HARDWARE -->
-        <xacro:property name="use_sim" value="false"/>
-        <ros2_control name="${name}" type="system">
-          <xacro:unless value="${use_sim}">
+        <ros2_control name="odrive_control" type="system">
             <hardware>
-              <plugin>odrive_ros2_control_plugin/ODriveHardwareInterface</plugin>
+              <!-- <plugin>odrive_ros2_control_plugin/ODriveHardwareInterface</plugin> -->
               <param name="can">can0</param>
+              <!-- <plugin>gazebo_ros2_control/GazeboSystem</plugin> -->
+              <plugin>mock_components/GenericSystem</plugin>
             </hardware>
-          </xacro:unless>
-          <xacro:if value="${use_sim}">
-            <hardware>
-              <!-- By default, set up controllers for simulation. This won't work on real hardware -->
-              <plugin>gazebo_ros2_control/GazeboSystem</plugin>
-              <!-- <plugin>mock_components/GenericSystem</plugin> -->
-          </hardware>
-          </xacro:if>
             <!-- JOINT DETAILS -->
             <joint name="shoulder_joint">
                 <command_interface name="position"/>
                 <state_interface name="position">
-                  <param name="initial_value">${initial_positions['shoulder_joint']}</param>
+                  <!-- <param name="initial_value">${initial_positions['shoulder_joint']}</param> -->
+                  <param name="initial_value">0.0</param>
                   <param name="node_id">0</param>
                 </state_interface>
@@ -31,5 +26,6 @@
                 <command_interface name="position"/>
                 <state_interface name="position">
-                  <param name="initial_value">${initial_positions['bicept_joint']}</param>
+                  <!-- <param name="initial_value">${initial_positions['bicept_joint']}</param> -->
+                  <param name="initial_value">0.0</param>
                   <param name="node_id">1</param>
                 </state_interface>
@@ -39,5 +35,6 @@
                 <command_interface name="position"/>
                 <state_interface name="position">
-                  <param name="initial_value">${initial_positions['elbow_joint']}</param>
+                  <!-- <param name="initial_value">${initial_positions['elbow_joint']}</param> -->
+                  <param name="initial_value">0.0</param>
                   <param name="node_id">2</param>
                 </state_interface>
@@ -47,5 +44,6 @@
                 <command_interface name="position"/>
                 <state_interface name="position">
-                  <param name="initial_value">${initial_positions['forearm_joint']}</param>
+                  <!-- <param name="initial_value">${initial_positions['forearm_joint']}</param> -->
+                  <param name="initial_value">0.0</param>
                   <param name="node_id">3</param>
                 </state_interface>
@@ -55,5 +53,6 @@
                 <command_interface name="position"/>
                 <state_interface name="position">
-                  <param name="initial_value">${initial_positions['wrist_joint1']}</param>
+                  <!-- <param name="initial_value">${initial_positions['wrist_joint1']}</param> -->
+                  <param name="initial_value">0.0</param>
                   <param name="node_id">4</param>
                 </state_interface>
@@ -63,5 +62,6 @@
                 <command_interface name="position"/>
                 <state_interface name="position">
-                  <param name="initial_value">${initial_positions['wrist_joint2']}</param>
+                  <!-- <param name="initial_value">${initial_positions['wrist_joint2']}</param> -->
+                  <param name="initial_value">0.0</param>
                   <param name="node_id">5</param>
                 </state_interface>
@@ -77,4 +77,4 @@
           </plugin>
       </gazebo>
-    </xacro:macro>
+    <!-- </xacro:macro> -->
 </robot>

File: src/moveit_config/config/robot.urdf.xacro (robot description, xacro)
@@ -3,7 +3,10 @@
     <xacro:arg name="initial_positions_file" default="initial_positions.yaml" />
     <!-- Import robot urdf file -->
-    <xacro:include filename="$(find arm_urdf)/description/arm.urdf" />
+    <xacro:include filename="$(find moveit_config)/config/robot_core.xacro" />
     <!-- Import control_xacro -->
-    <xacro:include filename="robot.ros2_control.xacro" />
-    <xacro:robot_ros2_control name="Gazebo" initial_positions_file="$(arg initial_positions_file)"/>
+    <xacro:include filename="$(find moveit_config)/config/robot.ros2_control.xacro" />
+    <!-- <xacro:robot_ros2_control name="Gazebo" initial_positions_file="$(arg initial_positions_file)"/> -->
+    <!-- <xacro:robot/> -->
+    <!-- <xacro:robot_ros2_control
+        name="odrive_control"/> -->
 </robot>
